Commit message: added active SLAM

File: description/gazebo_control.xacro (robot description, xacro)
@@ -4,6 +4,6 @@
         <plugin name="diff_drive" filename="libgazebo_ros_diff_drive.so">
             <!--WHEEL INFORMATION-->
-            <left_joint>left_wheel_joint</left_joint>
-            <right_joint>right_wheel_joint</right_joint>
+            <left_joint>left_rear</left_joint>
+            <right_joint>right_rear</right_joint>
             <wheel_separation>0.2</wheel_separation>
             <wheel_diameter>0.2</wheel_diameter>

File: description/robot.urdf.xacro (robot description, xacro)
@@ -1,7 +1,17 @@
 <?xml version="1.0"?>
 <robot xmlns:xacro="http://www.ros.org/wiki/xacro"  name="robot">
-    <xacro:include filename="robot_core.xacro"/>
+    <!--<xacro:include filename="robot_core.xacro"/>
     <xacro:include filename="lidar.xacro"/>
     <xacro:include filename="ros2_control.xacro"/>
-    <!--<xacro:include filename="imu.xacro"/>-->
+    <xacro:include filename="imu.xacro"/>-->
+    <xacro:arg name="use_ros2_control" default="true"/>
+    <xacro:arg name="sim_mode" default="false"/>
+    <xacro:include filename="robot_core.xacro" />
+    <xacro:if value="$(arg use_ros2_control)">
+        <xacro:include filename="ros2_control.xacro" />
+    </xacro:if>
+    <xacro:unless value="$(arg use_ros2_control)">
+        <xacro:include filename="gazebo_control.xacro" />
+    </xacro:unless>
+    <xacro:include filename="lidar.xacro" />
 </robot>

File: description/robot_core.xacro (robot description, xacro)
@@ -55,11 +55,11 @@
     </gazebo>
     <!--LEFT WHEEL LINK-->
-    <joint name="left_front" type="continuous">
+    <joint name="left_wheel_joint" type="continuous">
         <parent link="base_link"/>
-        <child link="left_wheel_rear"/>
+        <child link="left_wheel"/>
         <origin xyz="-0.0625 0.11 0" rpy="-${pi/2} 0 0"/>
         <axis xyz="0 0 1"/>
     </joint>
-    <link name="left_wheel_rear">
+    <link name="left_wheel">
         <visual>
             <geometry>
@@ -77,15 +77,15 @@
         </xacro:inertial_cylinder>
     </link>
-    <gazebo reference="left_wheel_rear">
+    <gazebo reference="left_wheel">
         <material>Gazebo/Black</material>
     </gazebo>
     <!--RIGHT REAR WHEEL-->
-    <joint name="right_front" type="continuous">
+    <joint name="right_wheel_joint" type="continuous">
         <parent link="base_link"/>
-        <child link="right_wheel_rear"/>
+        <child link="right_wheel"/>
         <origin xyz="-0.0625 -0.11 0" rpy="${pi/2} 0 0"/>
         <axis xyz="0 0 -1"/>
     </joint>
-    <link name="right_wheel_rear">
+    <link name="right_wheel">
         <visual>
             <geometry>
@@ -103,5 +103,5 @@
         </xacro:inertial_cylinder>
     </link>
-    <gazebo reference="right_wheel_rear">
+    <gazebo reference="right_wheel">
         <material>Gazebo/Black</material>
     </gazebo>
