Commit message: Hardware Integration Changes

File: description/robot_core.xacro (robot description, xacro)
@@ -37,5 +37,5 @@
             <origin xyz="0.125 0 0.05"/>
             <geometry>
-                <box size="0.25 0.2 0.1"/>
+                <box size="0.25 0.173 0.1"/>
             </geometry>
             <material name="white"/>
@@ -44,8 +44,8 @@
             <origin xyz="0.125 0 0.05"/>
             <geometry>
-                <box size="0.25 0.2 0.1"/>
+                <box size="0.25 0.173 0.1"/>
             </geometry>
         </collision>
-        <xacro:inertial_box mass="0.5" x="0.25" y="0.2" z="0.1" >
+        <xacro:inertial_box mass="0.5" x="0.25" y="0.173" z="0.1" >
             <origin xyz="0.125 0 0.05" rpy="0 0 0"/>
         </xacro:inertial_box>
@@ -58,5 +58,5 @@
         <parent link="base_link"/>
         <child link="left_wheel"/>
-        <origin xyz="-0.0625 0.11 0" rpy="-${pi/2} 0 0"/>
+        <origin xyz="-0.06255 0.0935 0" rpy="-${pi/2} 0 0"/>
         <axis xyz="0 0 1"/>
     </joint>
@@ -64,5 +64,5 @@
         <visual>
             <geometry>
-                <cylinder radius="0.05" length="0.02"/>
+                <cylinder radius="0.0325" length="0.02"/>
             </geometry>
             <material name="black"/>
@@ -70,8 +70,8 @@
         <collision>
             <geometry>
-                <cylinder radius="0.05" length="0.02"/>
+                <cylinder radius="0.0325" length="0.02"/>
             </geometry>
         </collision>
-        <xacro:inertial_cylinder mass="0.1" length="0.02" radius="0.05">
+        <xacro:inertial_cylinder mass="0.1" length="0.02" radius="0.0325">
             <origin xyz="0 0 0" rpy="0 0 0"/>
         </xacro:inertial_cylinder>
@@ -84,5 +84,5 @@
         <parent link="base_link"/>
         <child link="right_wheel"/>
-        <origin xyz="-0.0625 -0.11 0" rpy="${pi/2} 0 0"/>
+        <origin xyz="-0.0625 -0.0935 0" rpy="${pi/2} 0 0"/>
         <axis xyz="0 0 -1"/>
     </joint>
@@ -90,5 +90,5 @@
         <visual>
             <geometry>
-                <cylinder radius="0.05" length="0.02"/>
+                <cylinder radius="0.0325" length="0.02"/>
             </geometry>
             <material name="black"/>
@@ -96,8 +96,8 @@
         <collision>
             <geometry>
-                <cylinder radius="0.05" length="0.02"/>
+                <cylinder radius="0.0325" length="0.02"/>
             </geometry>
         </collision>
-        <xacro:inertial_cylinder mass="0.1" length="0.02" radius="0.05">
+        <xacro:inertial_cylinder mass="0.1" length="0.02" radius="0.0325">
             <origin xyz="0 0 0" rpy="0 0 0"/>
         </xacro:inertial_cylinder>
@@ -115,5 +115,5 @@
         <visual>
             <geometry>
-                <sphere radius="0.05"/>
+                <sphere radius="0.0325"/>
             </geometry>
             <material name="black"/>
@@ -121,8 +121,8 @@
         <collision>
             <geometry>
-                <sphere radius="0.05"/>
+                <sphere radius="0.0325"/>
             </geometry>
         </collision>
-        <xacro:inertial_sphere mass="0.1" radius="0.05">
+        <xacro:inertial_sphere mass="0.1" radius="0.0325">
             <origin xyz="0 0 0" rpy="0 0 0"/>
         </xacro:inertial_sphere>

File: description/ros2_control.xacro (robot description, xacro)
@@ -11,5 +11,5 @@
                 <param name="baud_rate">57600</param>
                 <param name="timeout">1000</param>
-                <param name="enc_counts_per_rev">3436</param>
+                <param name="enc_counts_per_rev">3960</param>
             </hardware>
             <joint name="left_wheel_joint">
