Commit message: Added ekfm, SLAM

File: description/lidar.xacro (robot description, xacro)
@@ -4,26 +4,27 @@
         <parent link="chassis"/>
         <child link="laser_frame"/>
-        <origin xyz="0.1 0 0.1" rpy="0 0 0"/>
+        <origin xyz="0.1 0 0.105" rpy="0 0 0"/>
     </joint>
     <link name="laser_frame">
         <visual>
             <geometry>
-                <cylinder radius="0.05" length="0.04"/>
+                <cylinder radius="0.05" length="0.05"/>
             </geometry>
-            <material name="red"/>
+            <material name="black"/>
         </visual>
         <collision>
             <geometry>
-                <cylinder radius="0.05" length="0.04"/>
+                <cylinder radius="0.05" length="0.05"/>
             </geometry>
         </collision>
-        <xacro:inertial_cylinder mass="0.1" length="0.04" radius="0.05">
+        <xacro:inertial_cylinder mass="0.1" length="0.05" radius="0.05">
             <origin xyz="0 0 0" rpy="0 0 0"/>
         </xacro:inertial_cylinder>
     </link>
-    <!--<gazebo reference="laser_frame">
+    <gazebo reference="laser_frame">
+        <material>Gazebo/Black</material>
         <sensor name="laser" type="ray">
             <pose>0 0 0 0 0 0</pose>
-            <visualize>true</visualize>
+            <visualize>false</visualize>
             <update_rate>10</update_rate>
             <ray>
@@ -50,4 +51,103 @@
             </plugin>
         </sensor>
-    </gazebo>-->
+    </gazebo>
+    <joint name="imu_joint" type="fixed">
+        <parent link="chassis"/>
+        <child link="imu_link"/>
+        <origin xyz="0.2 0 0.105"/>
+    </joint>
+    <link name="imu_link">
+        <visual>
+            <geometry>
+                <box size="0.05 0.05 0.01"/>
+            </geometry>
+            <material name="black"/>
+        </visual>
+        <collision>
+            <geometry>
+                <box size="0.05 0.05 0.01"/>
+            </geometry>
+        </collision>
+        <xacro:inertial_box mass="0.01" x="0.05" y="0.05" z="0.01">
+            <origin xyz="0 0 0" rpy="0 0 0"/>
+        </xacro:inertial_box>
+    </link>
+    <gazebo reference="imu_link">
+        <gravity>true</gravity>
+        <sensor name="bmb_imu" type="imu">
+            <always_on>true</always_on>
+            <update_rate>100</update_rate>
+            <visualize>true</visualize>
+            <imu>
+                <orientation>
+                    <x>
+                        <noise type="gaussian">
+                            <mean>0.0</mean>
+                            <stddev>2e-3</stddev>
+                        </noise>
+                    </x>
+                    <y>
+                        <noise type="gaussian">
+                            <mean>0.0</mean>
+                            <stddev>2e-3</stddev>
+                        </noise>
+                    </y>
+                    <z>
+                        <noise type="gaussian">
+                            <mean>0.0</mean>
+                            <stddev>2e-3</stddev>
+                        </noise>
+                    </z>
+                </orientation>
+                <angular_velocity>
+                    <x>
+                        <noise type="gaussian">
+                            <mean>0.0</mean>
+                            <stddev>2e-4</stddev>
+                        </noise>
+                    </x>
+                    <y>
+                        <noise type="gaussian">
+                            <mean>0.0</mean>
+                        <stddev>2e-4</stddev>
+                    </noise>
+                    </y>
+                    <z>
+                        <noise type="gaussian">
+                            <mean>0.0</mean>
+                            <stddev>2e-4</stddev>
+                        </noise>
+                    </z>
+                </angular_velocity>
+                <linear_acceleration>
+                    <x>
+                        <noise type="gaussian">
+                            <mean>0.0</mean>
+                            <stddev>1.7e-2</stddev>
+                        </noise>
+                    </x>
+                    <y>
+                        <noise type="gaussian">
+                            <mean>0.0</mean>
+                            <stddev>1.7e-2</stddev>
+                        </noise>
+                    </y>
+                    <z>
+                        <noise type="gaussian">
+                            <mean>0.0</mean>
+                            <stddev>1.7e-2</stddev>
+                        </noise>
+                    </z>
+                </linear_acceleration>
+            </imu>
+            <plugin name="basic_mobile_bot_imu" filename="libgazebo_ros_imu_sensor.so">
+                <initial_orientation_as_reference>false</initial_orientation_as_reference>
+                <frame_name>imu_link</frame_name>
+                <ros>
+                    <namespace>/imu</namespace>
+                    <remapping>~/out:=data</remapping>
+                </ros>
+            </plugin>
+        </sensor>
+    </gazebo>
 </robot>

File: description/robot.urdf.xacro (robot description, xacro)
@@ -3,3 +3,5 @@
     <xacro:include filename="robot_core.xacro"/>
     <xacro:include filename="lidar.xacro"/>
+    <xacro:include filename="ros2_control.xacro"/>
+    <!--<xacro:include filename="imu.xacro"/>-->
 </robot>

File: description/robot_core copy.xacro (robot description, xacro)
@@ -55,5 +55,30 @@
     </gazebo>
     <!--LEFT WHEEL LINK-->
-    <joint name="left_front" type="continuous">
+    <!--<joint name="left_front" type="continuous">
+        <parent link="base_link"/>
+        <child link="left_wheel_front"/>
+        <origin xyz="0.0625 0.11 0" rpy="-${pi/2} 0 0"/>
+        <axis xyz="0 0 1"/>
+    </joint>
+    <link name="left_wheel_front">
+        <visual>
+            <geometry>
+                <cylinder radius="0.05" length="0.02"/>
+            </geometry>
+            <material name="blue"/>
+        </visual>
+        <collision>
+            <geometry>
+                <cylinder radius="0.05" length="0.02"/>
+            </geometry>
+        </collision>
+        <xacro:inertial_cylinder mass="0.1" length="0.02" radius="0.05">
+            <origin xyz="0 0 0" rpy="0 0 0"/>
+        </xacro:inertial_cylinder>
+    </link>
+    <gazebo reference="left_wheel_front">
+        <material>Gazebo/Blue</material>
+    </gazebo>-->
+    <joint name="left_rear" type="continuous">
         <parent link="base_link"/>
         <child link="left_wheel_rear"/>
@@ -80,6 +105,32 @@
         <material>Gazebo/Black</material>
     </gazebo>
+    <!--RIGHT WHEEL LINK-->
+    <!--<joint name="right_front" type="continuous">
+        <parent link="base_link"/>
+        <child link="right_wheel_front"/>
+        <origin xyz="0.0625 -0.11 0" rpy="${pi/2} 0 0"/>
+        <axis xyz="0 0 -1"/>
+    </joint>
+    <link name="right_wheel_front">
+        <visual>
+            <geometry>
+                <cylinder radius="0.05" length="0.02"/>
+            </geometry>
+            <material name="blue"/>
+        </visual>
+        <collision>
+            <geometry>
+                <cylinder radius="0.05" length="0.02"/>
+            </geometry>
+        </collision>
+        <xacro:inertial_cylinder mass="0.1" length="0.02" radius="0.05">
+            <origin xyz="0 0 0" rpy="0 0 0"/>
+        </xacro:inertial_cylinder>
+    </link>
+    <gazebo reference="right_wheel_front">
+        <material>Gazebo/Blue</material>
+    </gazebo>-->
     <!--RIGHT REAR WHEEL-->
-    <joint name="right_front" type="continuous">
+    <joint name="right_rear" type="continuous">
         <parent link="base_link"/>
         <child link="right_wheel_rear"/>

Commit message: Changed Wheel Separation

File: description/lidar.xacro (robot description, xacro)
@@ -4,10 +4,10 @@
         <parent link="chassis"/>
         <child link="laser_frame"/>
-        <origin xyz="0.1 0 0.105" rpy="0 0 0"/>
+        <origin xyz="0.214 0 0.07" rpy="0 0 0"/>
     </joint>
     <link name="laser_frame">
         <visual>
             <geometry>
-                <cylinder radius="0.05" length="0.05"/>
+                <cylinder radius="0.025" length="0.03"/>
             </geometry>
             <material name="black"/>
@@ -15,8 +15,8 @@
         <collision>
             <geometry>
-                <cylinder radius="0.05" length="0.05"/>
+                <cylinder radius="0.025" length="0.03"/>
             </geometry>
         </collision>
-        <xacro:inertial_cylinder mass="0.1" length="0.05" radius="0.05">
+        <xacro:inertial_cylinder mass="0.3" length="0.03" radius="0.025">
             <origin xyz="0 0 0" rpy="0 0 0"/>
         </xacro:inertial_cylinder>
@@ -52,5 +52,5 @@
         </sensor>
     </gazebo>
-    <joint name="imu_joint" type="fixed">
+    <!--<joint name="imu_joint" type="fixed">
         <parent link="chassis"/>
         <child link="imu_link"/>
@@ -150,4 +150,4 @@
             </plugin>
         </sensor>
-    </gazebo>
+    </gazebo>-->
 </robot>

File: description/robot.urdf.xacro (robot description, xacro)
@@ -7,5 +7,5 @@
     <xacro:arg name="use_ros2_control" default="true"/>
     <xacro:arg name="sim_mode" default="true"/>
-    <xacro:include filename="robot_core_copy.xacro" />
+    <xacro:include filename="robot_core.xacro" />
     <xacro:if value="$(arg use_ros2_control)">
         <xacro:include filename="ros2_control.xacro" />

File: description/robot_core.xacro (robot description, xacro)
@@ -1,23 +1,38 @@
 <?xml version="1.0"?>
-<robot xmlns:xacro="http://www.ros.org/wiki/xacro"  name="robot">
+<robot xmlns:xacro="http://www.ros.org/wiki/xacro" >
     <xacro:include filename="inertial_macros.xacro"/>
+    <xacro:property name="chassis_length" value="0.25"/>
+    <xacro:property name="chassis_width" value="0.172"/>
+    <xacro:property name="chassis_height" value="0.07"/>
+    <xacro:property name="chassis_mass" value="1.7"/>
+    <xacro:property name="wheel_radius" value="0.0325"/>
+    <xacro:property name="wheel_thickness" value="0.012"/>
+    <xacro:property name="wheel_mass" value="0.05"/>
+    <xacro:property name="wheel_offset_x" value="0.193"/>
+    <xacro:property name="wheel_offset_y" value="0.092"/>
+    <xacro:property name="wheel_offset_z" value="0.01"/>
+    <xacro:property name="caster_wheel_radius" value="0.01"/>
+    <xacro:property name="caster_wheel_mass" value="0.01"/>
+    <xacro:property name="caster_wheel_offset_x" value="0.075"/>
+    <xacro:property name="caster_wheel_offset_z" value="${wheel_offset_z - wheel_radius + caster_wheel_radius}"/>
     <material name="white">
-        <color rgba='1 1 1 1'/>
+        <color rgba="1 1 1 1" />
     </material>
     <material name="orange">
-        <color rgba='1 0.3 0.1 1'/>
+        <color rgba="1 0.3 0.1 1"/>
     </material>
     <material name="blue">
-        <color rgba='0.2 0.2 1 1'/>
+        <color rgba="0.2 0.2 1 1"/>
     </material>
     <material name="black">
-        <color rgba='0 0 0 1'/>
+        <color rgba="0 0 0 1"/>
     </material>
     <material name="red">
-        <color rgba='1 0 0 1'/>
+        <color rgba="1 0 0 1"/>
     </material>
-    <!--BASE LINK-->
+    <!-- BASE LINK -->
     <link name="base_link">
     </link>
+    <!-- BASE_FOOTPRINT LINK -->
     <joint name="base_footprint_joint" type="fixed">
         <parent link="base_link"/>
@@ -27,36 +42,36 @@
     <link name="base_footprint">
     </link>
-    <!--CHASSIS LINK-->
+    <!-- CHASSIS LINK -->
     <joint name="chassis_joint" type="fixed">
         <parent link="base_link"/>
         <child link="chassis"/>
-        <origin xyz="-0.125 0 0"/>
+        <origin xyz="${-wheel_offset_x} 0 ${-wheel_offset_z}"/>
     </joint>
     <link name="chassis">
         <visual>
-            <origin xyz="0.125 0 0.05"/>
+            <origin xyz="${chassis_length/2} 0 ${chassis_height/2}"/>
             <geometry>
-                <box size="0.25 0.173 0.1"/>
+                <box size="${chassis_length} ${chassis_width} ${chassis_height}"/>
             </geometry>
-            <material name="white"/>
+            <material name="orange"/>
         </visual>
         <collision>
-            <origin xyz="0.125 0 0.05"/>
+            <origin xyz="${chassis_length/2} 0 ${chassis_height/2}"/>
             <geometry>
-                <box size="0.25 0.173 0.1"/>
+                <box size="${chassis_length} ${chassis_width} ${chassis_height}"/>
             </geometry>
         </collision>
-        <xacro:inertial_box mass="0.5" x="0.25" y="0.173" z="0.1" >
-            <origin xyz="0.125 0 0.05" rpy="0 0 0"/>
+        <xacro:inertial_box mass="0.5" x="${chassis_length}" y="${chassis_width}" z="${chassis_height}">
+            <origin xyz="${chassis_length/2} 0 ${chassis_height/2}" rpy="0 0 0"/>
         </xacro:inertial_box>
     </link>
     <gazebo reference="chassis">
-        <material>Gazebo/White</material>
+        <material>Gazebo/Orange</material>
     </gazebo>
-    <!--LEFT WHEEL LINK-->
+    <!-- LEFT WHEEL LINK -->
     <joint name="left_wheel_joint" type="continuous">
         <parent link="base_link"/>
         <child link="left_wheel"/>
-        <origin xyz="-0.06255 0.0935 0" rpy="-${pi/2} 0 0"/>
+        <origin xyz="0 ${wheel_offset_y} 0" rpy="-${pi/2} 0 0" />
         <axis xyz="0 0 1"/>
     </joint>
@@ -64,25 +79,25 @@
         <visual>
             <geometry>
-                <cylinder radius="0.0325" length="0.02"/>
+                <cylinder radius="${wheel_radius}" length="${wheel_thickness}"/>
             </geometry>
-            <material name="black"/>
+            <material name="blue"/>
         </visual>
         <collision>
             <geometry>
-                <cylinder radius="0.0325" length="0.02"/>
+                <sphere radius="${wheel_radius}"/>
             </geometry>
         </collision>
-        <xacro:inertial_cylinder mass="0.1" length="0.02" radius="0.0325">
+        <xacro:inertial_cylinder mass="${wheel_mass}" length="${wheel_thickness}" radius="${wheel_radius}">
             <origin xyz="0 0 0" rpy="0 0 0"/>
         </xacro:inertial_cylinder>
     </link>
     <gazebo reference="left_wheel">
-        <material>Gazebo/Black</material>
+        <material>Gazebo/Blue</material>
     </gazebo>
-    <!--RIGHT REAR WHEEL-->
+    <!-- RIGHT WHEEL LINK -->
     <joint name="right_wheel_joint" type="continuous">
         <parent link="base_link"/>
         <child link="right_wheel"/>
-        <origin xyz="-0.0625 -0.0935 0" rpy="${pi/2} 0 0"/>
+        <origin xyz="0 ${-wheel_offset_y} 0" rpy="${pi/2} 0 0" />
         <axis xyz="0 0 -1"/>
     </joint>
@@ -90,44 +105,44 @@
         <visual>
             <geometry>
-                <cylinder radius="0.0325" length="0.02"/>
+                <cylinder radius="${wheel_radius}" length="${wheel_thickness}"/>
             </geometry>
-            <material name="black"/>
+            <material name="blue"/>
         </visual>
         <collision>
             <geometry>
-                <cylinder radius="0.0325" length="0.02"/>
+                <sphere radius="${wheel_radius}"/>
             </geometry>
         </collision>
-        <xacro:inertial_cylinder mass="0.1" length="0.02" radius="0.0325">
+        <xacro:inertial_cylinder mass="${wheel_mass}" length="${wheel_thickness}" radius="${wheel_radius}">
             <origin xyz="0 0 0" rpy="0 0 0"/>
         </xacro:inertial_cylinder>
     </link>
     <gazebo reference="right_wheel">
-        <material>Gazebo/Black</material>
+        <material>Gazebo/Blue</material>
     </gazebo>
+    <!-- CASTER WHEEL LINK -->
     <joint name="caster_wheel_joint" type="fixed">
-        <parent link="base_link"/>
+        <parent link="chassis"/>
         <child link="caster_wheel"/>
-        <origin xyz="0.0625 0. 0" rpy="0 0 0"/>
-        <axis xyz="0 0 1"/>
+        <origin xyz="${caster_wheel_offset_x} 0 ${caster_wheel_offset_z}"/>
     </joint>
     <link name="caster_wheel">
         <visual>
             <geometry>
-                <sphere radius="0.0325"/>
+                <sphere radius="${caster_wheel_radius}"/>
             </geometry>
-            <material name="black"/>
+            <material name="white"/>
         </visual>
         <collision>
             <geometry>
-                <sphere radius="0.0325"/>
+                <sphere radius="${caster_wheel_radius}"/>
             </geometry>
         </collision>
-        <xacro:inertial_sphere mass="0.1" radius="0.0325">
+        <xacro:inertial_sphere mass="${caster_wheel_mass}" radius="${caster_wheel_radius}">
             <origin xyz="0 0 0" rpy="0 0 0"/>
         </xacro:inertial_sphere>
     </link>
     <gazebo reference="caster_wheel">
-        <material>Gazebo/Black</material>
+        <material>Gazebo/White</material>
         <mu1 value="0.001"/>
         <mu2 value="0.001"/>

File: description/ros2_control.xacro (robot description, xacro)
@@ -5,6 +5,6 @@
             <hardware>
                 <plugin>diffdrive_arduino/DiffDriveArduino</plugin>
-                <param name="left_wheel_name">left_rear</param>
-                <param name="right_wheel_name">right_rear</param>
+                <param name="left_wheel_name">left_wheel_joint</param>
+                <param name="right_wheel_name">right_wheel_joint</param>
                 <param name="loop_rate">30</param>
                 <param name="device">/dev/ttyUSB0</param>
@@ -13,5 +13,5 @@
                 <param name="enc_counts_per_rev">3960</param>
             </hardware>
-            <joint name="left_rear">
+            <joint name="left_wheel_joint">
                 <command_interface name="velocity">
                     <param name="min">-10</param>
@@ -21,5 +21,5 @@
                 <state_interface name="position"/>
             </joint>
-            <joint name="right_rear">
+            <joint name="right_wheel_joint">
                 <command_interface name="velocity">
                     <param name="min">-10</param>
@@ -36,5 +36,5 @@
                 <plugin>gazebo_ros2_control/GazeboSystem</plugin>
             </hardware>
-            <joint name="left_rear">
+            <joint name="left_wheel_joint">
                 <command_interface name="velocity">
                     <param name="min">-10</param>
@@ -44,21 +44,5 @@
                 <state_interface name="position"/>
             </joint>
-            <joint name="right_rear">
-                <command_interface name="velocity">
-                    <param name="min">-10</param>
-                    <param name="max">10</param>
-                </command_interface>
-                <state_interface name="velocity"/>
-                <state_interface name="position"/>
-            </joint>
-            <joint name="left_front">
-                <command_interface name="velocity">
-                    <param name="min">-10</param>
-                    <param name="max">10</param>
-                </command_interface>
-                <state_interface name="velocity"/>
-                <state_interface name="position"/>
-            </joint>
-            <joint name="right_front">
+            <joint name="right_wheel_joint">
                 <command_interface name="velocity">
                     <param name="min">-10</param>
