Commit message: added hardware compatibility

File: description/robot.urdf.xacro (robot description, xacro)
@@ -5,6 +5,6 @@
     <xacro:include filename="ros2_control.xacro"/>
     <xacro:include filename="imu.xacro"/>-->
-    <xacro:arg name="use_ros2_control" default="false"/>
-    <xacro:arg name="sim_mode" default="true"/>
+    <xacro:arg name="use_ros2_control" default="true"/>
+    <xacro:arg name="sim_mode" default="false"/>
     <xacro:include filename="robot_core.xacro" />
     <xacro:if value="$(arg use_ros2_control)">

File: description/ros2_control.xacro (robot description, xacro)
@@ -1,29 +1,61 @@
 <?xml version="1.0"?>
 <robot xmlns:xacro="http://www.ros.org/wiki/xacro">
-    <ros2_control name="GazeboSystem" type="system">
-        <hardware>
-            <plugin>gazebo_ros2_control/GazeboSystem</plugin>
-        </hardware>
-        <joint name="left_wheel_joint">
-            <command_interface name="velocity">
-                <param name="min">-10</param>
-                <param name="max">10</param>
-            </command_interface>
-            <state_interface name="velocity"/>
-            <state_interface name="position"/>
-        </joint>
-        <joint name="right_wheel_joint">
-            <command_interface name="velocity">
-                <param name="min">-10</param>
-                <param name="max">10</param>
-            </command_interface>
-            <state_interface name="velocity"/>
-            <state_interface name="position"/>
-        </joint>
-    </ros2_control>
+    <xacro:unless value="$(arg sim_mode)">
+        <ros2_control name="RealRobot" type="system">
+            <hardware>
+                <plugin>diffdrive_arduino/DiffDriveArduino</plugin>
+                <param name="left_wheel_name">left_wheel_joint</param>
+                <param name="right_wheel_name">right_wheel_joint</param>
+                <param name="loop_rate">30</param>
+                <param name="device">/dev/ttyUSB0</param>
+                <param name="baud_rate">57600</param>
+                <param name="timeout">1000</param>
+                <param name="enc_counts_per_rev">3436</param>
+            </hardware>
+            <joint name="left_wheel_joint">
+                <command_interface name="velocity">
+                    <param name="min">-10</param>
+                    <param name="max">10</param>
+                </command_interface>
+                <state_interface name="velocity"/>
+                <state_interface name="position"/>
+            </joint>
+            <joint name="right_wheel_joint">
+                <command_interface name="velocity">
+                    <param name="min">-10</param>
+                    <param name="max">10</param>
+                </command_interface>
+                <state_interface name="velocity"/>
+                <state_interface name="position"/>
+            </joint>
+        </ros2_control>
+    </xacro:unless>
+    <xacro:if value="$(arg sim_mode)">
+        <ros2_control name="GazeboSystem" type="system">
+            <hardware>
+                <plugin>gazebo_ros2_control/GazeboSystem</plugin>
+            </hardware>
+            <joint name="left_wheel_joint">
+                <command_interface name="velocity">
+                    <param name="min">-10</param>
+                    <param name="max">10</param>
+                </command_interface>
+                <state_interface name="velocity"/>
+                <state_interface name="position"/>
+            </joint>
+            <joint name="right_wheel_joint">
+                <command_interface name="velocity">
+                    <param name="min">-10</param>
+                    <param name="max">10</param>
+                </command_interface>
+                <state_interface name="velocity"/>
+                <state_interface name="position"/>
+            </joint>
+        </ros2_control>
+    </xacro:if>
     <gazebo>
         <plugin name="gazebo_ros2_control" filename="libgazebo_ros2_control.so">
-            <parameters>$(find vander_one)/config/my_controllers.yaml</parameters>
-            <parameters>$(find vander_one)/config/gaz_ros2_ctl_use_sim.yaml</parameters>
+            <parameters>$(find articubot_one)/config/my_controllers.yaml</parameters>
+            <parameters>$(find articubot_one)/config/gaz_ros2_ctl_use_sim.yaml</parameters>
         </plugin>
     </gazebo>

Commit message: Hardware changes

File: description/robot.urdf.xacro (robot description, xacro)
@@ -6,6 +6,6 @@
     <xacro:include filename="imu.xacro"/>-->
     <xacro:arg name="use_ros2_control" default="true"/>
-    <xacro:arg name="sim_mode" default="false"/>
-    <xacro:include filename="robot_core.xacro" />
+    <xacro:arg name="sim_mode" default="true"/>
+    <xacro:include filename="robot_core_copy.xacro" />
     <xacro:if value="$(arg use_ros2_control)">
         <xacro:include filename="ros2_control.xacro" />

File: description/robot_core_copy.xacro (robot description, xacro)
@@ -37,5 +37,5 @@
             <origin xyz="0.125 0 0.05"/>
             <geometry>
-                <box size="0.25 0.2 0.1"/>
+                <box size="0.25 0.173 0.1"/>
             </geometry>
             <material name="white"/>
@@ -44,8 +44,8 @@
             <origin xyz="0.125 0 0.05"/>
             <geometry>
-                <box size="0.25 0.2 0.1"/>
+                <box size="0.25 0.173 0.1"/>
             </geometry>
         </collision>
-        <xacro:inertial_box mass="0.5" x="0.25" y="0.2" z="0.1" >
+        <xacro:inertial_box mass="0.5" x="0.25" y="0.173" z="0.1" >
             <origin xyz="0.125 0 0.05" rpy="0 0 0"/>
         </xacro:inertial_box>
@@ -55,8 +55,8 @@
     </gazebo>
     <!--LEFT WHEEL LINK-->
-    <!--<joint name="left_front" type="continuous">
+    <joint name="left_front" type="continuous">
         <parent link="base_link"/>
         <child link="left_wheel_front"/>
-        <origin xyz="0.0625 0.11 0" rpy="-${pi/2} 0 0"/>
+        <origin xyz="0.065 0.086 0" rpy="-${pi/2} 0 0"/>
         <axis xyz="0 0 1"/>
     </joint>
@@ -64,5 +64,5 @@
         <visual>
             <geometry>
-                <cylinder radius="0.05" length="0.02"/>
+                <cylinder radius="0.0325" length="0.02"/>
             </geometry>
             <material name="blue"/>
@@ -70,8 +70,8 @@
         <collision>
             <geometry>
-                <cylinder radius="0.05" length="0.02"/>
+                <cylinder radius="0.0325" length="0.02"/>
             </geometry>
         </collision>
-        <xacro:inertial_cylinder mass="0.1" length="0.02" radius="0.05">
+        <xacro:inertial_cylinder mass="0.1" length="0.02" radius="0.0325">
             <origin xyz="0 0 0" rpy="0 0 0"/>
         </xacro:inertial_cylinder>
@@ -79,9 +79,9 @@
     <gazebo reference="left_wheel_front">
         <material>Gazebo/Blue</material>
-    </gazebo>-->
+    </gazebo>
     <joint name="left_rear" type="continuous">
         <parent link="base_link"/>
         <child link="left_wheel_rear"/>
-        <origin xyz="-0.0625 0.11 0" rpy="-${pi/2} 0 0"/>
+        <origin xyz="-0.065 0.086 0" rpy="-${pi/2} 0 0"/>
         <axis xyz="0 0 1"/>
     </joint>
@@ -89,5 +89,5 @@
         <visual>
             <geometry>
-                <cylinder radius="0.05" length="0.02"/>
+                <cylinder radius="0.0325" length="0.02"/>
             </geometry>
             <material name="black"/>
@@ -95,8 +95,8 @@
         <collision>
             <geometry>
-                <cylinder radius="0.05" length="0.02"/>
+                <cylinder radius="0.0325" length="0.02"/>
             </geometry>
         </collision>
-        <xacro:inertial_cylinder mass="0.1" length="0.02" radius="0.05">
+        <xacro:inertial_cylinder mass="0.1" length="0.02" radius="0.0325">
             <origin xyz="0 0 0" rpy="0 0 0"/>
         </xacro:inertial_cylinder>
@@ -106,8 +106,8 @@
     </gazebo>
     <!--RIGHT WHEEL LINK-->
-    <!--<joint name="right_front" type="continuous">
+    <joint name="right_front" type="continuous">
         <parent link="base_link"/>
         <child link="right_wheel_front"/>
-        <origin xyz="0.0625 -0.11 0" rpy="${pi/2} 0 0"/>
+        <origin xyz="0.065 -0.086 0" rpy="${pi/2} 0 0"/>
         <axis xyz="0 0 -1"/>
     </joint>
@@ -115,5 +115,5 @@
         <visual>
             <geometry>
-                <cylinder radius="0.05" length="0.02"/>
+                <cylinder radius="0.0325" length="0.02"/>
             </geometry>
             <material name="blue"/>
@@ -121,8 +121,8 @@
         <collision>
             <geometry>
-                <cylinder radius="0.05" length="0.02"/>
+                <cylinder radius="0.0325" length="0.02"/>
             </geometry>
         </collision>
-        <xacro:inertial_cylinder mass="0.1" length="0.02" radius="0.05">
+        <xacro:inertial_cylinder mass="0.1" length="0.02" radius="0.0325">
             <origin xyz="0 0 0" rpy="0 0 0"/>
         </xacro:inertial_cylinder>
@@ -130,10 +130,10 @@
     <gazebo reference="right_wheel_front">
         <material>Gazebo/Blue</material>
-    </gazebo>-->
+    </gazebo>
     <!--RIGHT REAR WHEEL-->
     <joint name="right_rear" type="continuous">
         <parent link="base_link"/>
         <child link="right_wheel_rear"/>
-        <origin xyz="-0.0625 -0.11 0" rpy="${pi/2} 0 0"/>
+        <origin xyz="-0.065 -0.086 0" rpy="${pi/2} 0 0"/>
         <axis xyz="0 0 -1"/>
     </joint>
@@ -141,5 +141,5 @@
         <visual>
             <geometry>
-                <cylinder radius="0.05" length="0.02"/>
+                <cylinder radius="0.0325" length="0.02"/>
             </geometry>
             <material name="black"/>
@@ -147,8 +147,8 @@
         <collision>
             <geometry>
-                <cylinder radius="0.05" length="0.02"/>
+                <cylinder radius="0.0325" length="0.02"/>
             </geometry>
         </collision>
-        <xacro:inertial_cylinder mass="0.1" length="0.02" radius="0.05">
+        <xacro:inertial_cylinder mass="0.1" length="0.02" radius="0.0325">
             <origin xyz="0 0 0" rpy="0 0 0"/>
         </xacro:inertial_cylinder>
@@ -157,5 +157,5 @@
         <material>Gazebo/Black</material>
     </gazebo>
-    <joint name="caster_wheel_joint" type="fixed">
+    <!--<joint name="caster_wheel_joint" type="fixed">
         <parent link="base_link"/>
         <child link="caster_wheel"/>
@@ -183,4 +183,4 @@
         <mu1 value="0.001"/>
         <mu2 value="0.001"/>
-    </gazebo>
+    </gazebo>-->
 </robot>

File: description/ros2_control.xacro (robot description, xacro)
@@ -5,6 +5,6 @@
             <hardware>
                 <plugin>diffdrive_arduino/DiffDriveArduino</plugin>
-                <param name="left_wheel_name">left_wheel_joint</param>
-                <param name="right_wheel_name">right_wheel_joint</param>
+                <param name="left_wheel_name">left_rear</param>
+                <param name="right_wheel_name">right_rear</param>
                 <param name="loop_rate">30</param>
                 <param name="device">/dev/ttyUSB0</param>
@@ -13,5 +13,5 @@
                 <param name="enc_counts_per_rev">3960</param>
             </hardware>
-            <joint name="left_wheel_joint">
+            <joint name="left_rear">
                 <command_interface name="velocity">
                     <param name="min">-10</param>
@@ -21,5 +21,5 @@
                 <state_interface name="position"/>
             </joint>
-            <joint name="right_wheel_joint">
+            <joint name="right_rear">
                 <command_interface name="velocity">
                     <param name="min">-10</param>
@@ -36,5 +36,5 @@
                 <plugin>gazebo_ros2_control/GazeboSystem</plugin>
             </hardware>
-            <joint name="left_wheel_joint">
+            <joint name="left_rear">
                 <command_interface name="velocity">
                     <param name="min">-10</param>
@@ -44,5 +44,21 @@
                 <state_interface name="position"/>
             </joint>
-            <joint name="right_wheel_joint">
+            <joint name="right_rear">
+                <command_interface name="velocity">
+                    <param name="min">-10</param>
+                    <param name="max">10</param>
+                </command_interface>
+                <state_interface name="velocity"/>
+                <state_interface name="position"/>
+            </joint>
+            <joint name="left_front">
+                <command_interface name="velocity">
+                    <param name="min">-10</param>
+                    <param name="max">10</param>
+                </command_interface>
+                <state_interface name="velocity"/>
+                <state_interface name="position"/>
+            </joint>
+            <joint name="right_front">
                 <command_interface name="velocity">
                     <param name="min">-10</param>
@@ -56,6 +72,6 @@
     <gazebo>
         <plugin name="gazebo_ros2_control" filename="libgazebo_ros2_control.so">
-            <parameters>$(find articubot_one)/config/my_controllers.yaml</parameters>
-            <parameters>$(find articubot_one)/config/gaz_ros2_ctl_use_sim.yaml</parameters>
+            <parameters>$(find vander_one)/config/my_controllers.yaml</parameters>
+            <parameters>$(find vander_one)/config/gaz_ros2_ctl_use_sim.yaml</parameters>
         </plugin>
     </gazebo>

Commit message: Changed Robot URDF

File: description/robot.urdf.xacro (robot description, xacro)
@@ -7,7 +7,7 @@
     <xacro:arg name="use_ros2_control" default="true"/>
     <xacro:arg name="sim_mode" default="true"/>
-    <xacro:include filename="robot_core.xacro" />
+    <xacro:include filename="robot_core1.xacro" />
     <xacro:if value="$(arg use_ros2_control)">
-        <xacro:include filename="ros2_control.xacro" />
+        <xacro:include filename="ros2_control1.xacro" />
     </xacro:if>
     <xacro:unless value="$(arg use_ros2_control)">

File: description/robot_core1.xacro (robot description, xacro)
@@ -70,57 +70,107 @@
     </gazebo>
     <!-- LEFT WHEEL LINK -->
-    <joint name="left_wheel_joint" type="continuous">
-        <parent link="base_link"/>
-        <child link="left_wheel"/>
+    <joint name="left_rear" type="continuous">
+        <parent link="base_link"/>
+        <child link="left_wheel_rear"/>
         <origin xyz="0 ${wheel_offset_y} 0" rpy="-${pi/2} 0 0" />
         <axis xyz="0 0 1"/>
     </joint>
-    <link name="left_wheel">
-        <visual>
-            <geometry>
-                <cylinder radius="${wheel_radius}" length="${wheel_thickness}"/>
-            </geometry>
-            <material name="blue"/>
-        </visual>
-        <collision>
-            <geometry>
-                <sphere radius="${wheel_radius}"/>
-            </geometry>
-        </collision>
-        <xacro:inertial_cylinder mass="${wheel_mass}" length="${wheel_thickness}" radius="${wheel_radius}">
-            <origin xyz="0 0 0" rpy="0 0 0"/>
-        </xacro:inertial_cylinder>
-    </link>
-    <gazebo reference="left_wheel">
+    <link name="left_wheel_rear">
+        <visual>
+            <geometry>
+                <cylinder radius="${wheel_radius}" length="${wheel_thickness}"/>
+            </geometry>
+            <material name="blue"/>
+        </visual>
+        <collision>
+            <geometry>
+                <sphere radius="${wheel_radius}"/>
+            </geometry>
+        </collision>
+        <xacro:inertial_cylinder mass="${wheel_mass}" length="${wheel_thickness}" radius="${wheel_radius}">
+            <origin xyz="0 0 0" rpy="0 0 0"/>
+        </xacro:inertial_cylinder>
+    </link>
+    <gazebo reference="left_wheel_rear">
+        <material>Gazebo/Blue</material>
+    </gazebo>
+    <joint name="left_front" type="continuous">
+        <parent link="base_link"/>
+        <child link="left_wheel_front"/>
+        <origin xyz="0.125 ${wheel_offset_y} 0" rpy="-${pi/2} 0 0" />
+        <axis xyz="0 0 1"/>
+    </joint>
+    <link name="left_wheel_front">
+        <visual>
+            <geometry>
+                <cylinder radius="${wheel_radius}" length="${wheel_thickness}"/>
+            </geometry>
+            <material name="blue"/>
+        </visual>
+        <collision>
+            <geometry>
+                <sphere radius="${wheel_radius}"/>
+            </geometry>
+        </collision>
+        <xacro:inertial_cylinder mass="${wheel_mass}" length="${wheel_thickness}" radius="${wheel_radius}">
+            <origin xyz="0 0 0" rpy="0 0 0"/>
+        </xacro:inertial_cylinder>
+    </link>
+    <gazebo reference="left_wheel_front">
         <material>Gazebo/Blue</material>
     </gazebo>
     <!-- RIGHT WHEEL LINK -->
-    <joint name="right_wheel_joint" type="continuous">
-        <parent link="base_link"/>
-        <child link="right_wheel"/>
+    <joint name="right_rear" type="continuous">
+        <parent link="base_link"/>
+        <child link="right_wheel_rear"/>
         <origin xyz="0 ${-wheel_offset_y} 0" rpy="${pi/2} 0 0" />
         <axis xyz="0 0 -1"/>
     </joint>
-    <link name="right_wheel">
-        <visual>
-            <geometry>
-                <cylinder radius="${wheel_radius}" length="${wheel_thickness}"/>
-            </geometry>
-            <material name="blue"/>
-        </visual>
-        <collision>
-            <geometry>
-                <sphere radius="${wheel_radius}"/>
-            </geometry>
-        </collision>
-        <xacro:inertial_cylinder mass="${wheel_mass}" length="${wheel_thickness}" radius="${wheel_radius}">
-            <origin xyz="0 0 0" rpy="0 0 0"/>
-        </xacro:inertial_cylinder>
-    </link>
-    <gazebo reference="right_wheel">
+    <link name="right_wheel_rear">
+        <visual>
+            <geometry>
+                <cylinder radius="${wheel_radius}" length="${wheel_thickness}"/>
+            </geometry>
+            <material name="blue"/>
+        </visual>
+        <collision>
+            <geometry>
+                <sphere radius="${wheel_radius}"/>
+            </geometry>
+        </collision>
+        <xacro:inertial_cylinder mass="${wheel_mass}" length="${wheel_thickness}" radius="${wheel_radius}">
+            <origin xyz="0 0 0" rpy="0 0 0"/>
+        </xacro:inertial_cylinder>
+    </link>
+    <gazebo reference="right_wheel_rear">
+        <material>Gazebo/Blue</material>
+    </gazebo>
+    <joint name="right_front" type="continuous">
+        <parent link="base_link"/>
+        <child link="right_wheel_front"/>
+        <origin xyz="0.125 ${-wheel_offset_y} 0" rpy="${pi/2} 0 0" />
+        <axis xyz="0 0 -1"/>
+    </joint>
+    <link name="right_wheel_front">
+        <visual>
+            <geometry>
+                <cylinder radius="${wheel_radius}" length="${wheel_thickness}"/>
+            </geometry>
+            <material name="blue"/>
+        </visual>
+        <collision>
+            <geometry>
+                <sphere radius="${wheel_radius}"/>
+            </geometry>
+        </collision>
+        <xacro:inertial_cylinder mass="${wheel_mass}" length="${wheel_thickness}" radius="${wheel_radius}">
+            <origin xyz="0 0 0" rpy="0 0 0"/>
+        </xacro:inertial_cylinder>
+    </link>
+    <gazebo reference="right_wheel_front">
         <material>Gazebo/Blue</material>
     </gazebo>
     <!-- CASTER WHEEL LINK -->
-    <joint name="caster_wheel_joint" type="fixed">
+    <!--<joint name="caster_wheel_joint" type="fixed">
         <parent link="chassis"/>
         <child link="caster_wheel"/>
@@ -147,4 +197,4 @@
         <mu1 value="0.001"/>
         <mu2 value="0.001"/>
-    </gazebo>
+    </gazebo>-->
 </robot>

File: description/ros2_control1.xacro (robot description, xacro)
@@ -5,6 +5,6 @@
             <hardware>
                 <plugin>diffdrive_arduino/DiffDriveArduino</plugin>
-                <param name="left_wheel_name">left_rear</param>
-                <param name="right_wheel_name">right_rear</param>
+                <param name="left_wheel_name">right_wheel_joint</param>
+                <param name="right_wheel_name">left_wheel_joint</param>
                 <param name="loop_rate">30</param>
                 <param name="device">/dev/ttyUSB0</param>
@@ -22,4 +22,20 @@
             </joint>
             <joint name="right_rear">
+                <command_interface name="velocity">
+                    <param name="min">-10</param>
+                    <param name="max">10</param>
+                </command_interface>
+                <state_interface name="velocity"/>
+                <state_interface name="position"/>
+            </joint>
+            <joint name="left_front">
+                <command_interface name="velocity">
+                    <param name="min">-10</param>
+                    <param name="max">10</param>
+                </command_interface>
+                <state_interface name="velocity"/>
+                <state_interface name="position"/>
+            </joint>
+            <joint name="right_front">
                 <command_interface name="velocity">
                     <param name="min">-10</param>
